File: Hardware/SparkX_EZ_Power_AAA.sch (EAGLE design)
At the start: 34 parts, among them J3 AVR_SPI_PROG_3X2TESTPOINTS, U1 ATTINY43_QFN20, U2 TPS61200

Commit message: Post-review updates
Parts:
- added RXD, TXD: TEST-POINT3X4, SparkFun-Connectors:TEST-POINT3X4
- C1: device SparkFun-Capacitors:10UF-0603-6.3V-20% -> SparkFun-Capacitors:10UF-0402T-6.3V-20%
- C2, C4, C6: device SparkFun-Capacitors:0.1UF-0402-10V-10%-X7R -> SparkFun-Capacitors:0.1UF-0402T-6.3V-10%-X7R
- L2: device SparkFun:INDUCTOR. -> SparkFun-Coils:4.7μH_SHIELDED_INDUCTOR
- R1: device SparkFun-Resistors:1MOHM-0603-1/4W-5% -> New-Parts_SparkFun-Resistors:1MOHM-0402T-1/16W-1%
- R2: device SparkFun-Resistors:180KOHM-0603-1/10W-1% -> New-Parts_SparkFun-Resistors:180KOHM-0402T-1/16W-1%
- R3: device SparkFun-Resistors:453KOHM-0603-1/10W-1% -> New-Parts_SparkFun-Resistors:453KOHM-0402T-1/16W-1%
- U2: device SparkFun:TPS61200 -> SparkFun-IC-Power:TPS61200_MINIMAL
Connections:
- new net RXD: RXD.1, U1.RXD/D13
- new net TXD: TXD.1, U1.TXD/D12
- net GND: no longer U2.PAD@1, U2.PAD@2, U2.PAD@3, U2.PAD@4, U2.PAD@5, U2.PGND
Other:
- moved on the sheet: 3V3_EN, C3, C4, C6, R1, R2

Commit message: Post-review updates
Parts:
- L2: value 4.7uH, 1.2A -> 4.7μH; device SparkFun-Coils:4.7μH_SHIELDED_INDUCTOR -> SparkFun-Coils:4.7μH_SHIELDED_INDUCTORNPIS_LS
Changed lines of the file:
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@@
 <setting verticaltext="up"/>
 </settings>
-<grid distance="0.1" unitdist="inch" unit="inch" style="lines" multiple="1" display="no" altdistance="0.01" altunitdist="inch" altunit="inch"/>
+<grid distance="0.1" unitdist="inch" unit="inch" style="lines" multiple="1" display="no" altdistance="0.05" altunitdist="inch" altunit="inch"/>
 <layers>
 <layer number="1" name="Top" color="4" fill="1" visible="no" active="no"/>
@@
 <part name="GND2" library="SparkFun-PowerSymbols" deviceset="GND" device=""/>
 <part name="C1" library="SparkFun-Capacitors" deviceset="10UF" device="-0402T-6.3V-20%" value="10uF"/>
-<part name="L2" library="SparkFun-Coils" deviceset="4.7μH_SHIELDED_INDUCTOR" device="" value="4.7uH, 1.2A"/>
+<part name="L2" library="SparkFun-Coils" deviceset="4.7μH_SHIELDED_INDUCTOR" device="NPIS_LS" value="4.7μH"/>
 <part name="SUPPLY1" library="SparkFun-PowerSymbols" deviceset="3.3V" device=""/>
 <part name="GND3" library="SparkFun-PowerSymbols" deviceset="GND" device=""/>

Commit message: Add VIN Max 5.5V
Parts:
- U1: device New-Parts_SparkFun-IC-Microcontroller:ATTINY43_QFN20 -> SparkFun-IC-Microcontroller:ATTINY43_QFN20
Other:
- note added: "Recommended VIN (Min) : 1.5V (1 x AAA) Recommended VIN (Max): 3.0V (2 x AAA) Maximum VIN: 5.5V"
- note removed: "Recommended VIN (Min) : 1.1V Recommended VIN (Max): 3.0V (2 x AAA)"
Changed lines of the file:
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@@
 <part name="PROC_PWR_EN" library="SparkFun-Jumpers" deviceset="JUMPER-SMT_2_NC_TRACE" device="_SILK" package3d_urn="urn:adsk.eagle:package:39281/1"/>
 <part name="3V3_EN" library="SparkFun-Connectors" deviceset="TEST-POINT" device="3X4" value="TEST-POINT3X4"/>
-<part name="U1" library="New-Parts_SparkFun-IC-Microcontroller" deviceset="ATTINY43" device="_QFN20"/>
+<part name="U1" library="SparkFun-IC-Microcontroller" deviceset="ATTINY43" device="_QFN20"/>
 <part name="SUPPLY11" library="SparkFun-PowerSymbols" deviceset="VIN" device=""/>
 <part name="GND7" library="SparkFun-PowerSymbols" deviceset="GND" device=""/>
@@
 <text x="261.62" y="152.654" size="1.778" layer="97">UVLO 1.0V</text>
 <text x="164.084" y="268.732" size="5.08" layer="94">Boost Converter</text>
-<text x="218.44" y="182.88" size="1.778" layer="97" ratio="15">Recommended VIN (Min) : 1.1V
-Recommended VIN (Max): 3.0V (2 x AAA)</text>
+<text x="218.44" y="182.88" size="1.778" layer="97" ratio="15">Recommended VIN (Min) : 1.5V (1 x AAA)
+Recommended VIN (Max): 3.0V (2 x AAA)
+Maximum VIN: 5.5V</text>
 <text x="218.44" y="195.58" size="1.778" layer="97" ratio="15">Caution!
 =====

Commit message: Update 16-way FPC Connector. Add missing PROD_IDs
Parts:
- IN, OUT: value FPC_16_0.5MM_BACKFLIP -> (none); device New_Parts_Connectors:FPC_16_0.5MM_BACKFLIP -> SparkFun-Connectors:CONN_16FPC_16_0.5MM
- R1: device New-Parts_SparkFun-Resistors:1MOHM-0402T-1/16W-1% -> SparkFun-Resistors:1MOHM-0402T-1/16W-5%
- R2: device New-Parts_SparkFun-Resistors:180KOHM-0402T-1/16W-1% -> SparkFun-Resistors:180KOHM-0402T-1/16W-1%
- R3: device New-Parts_SparkFun-Resistors:453KOHM-0402T-1/16W-1% -> SparkFun-Resistors:453KOHM-0402T-1/16W-1%
Changed lines of the file:
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@@
 <part name="FD3" library="SparkFun-Aesthetics" deviceset="FIDUCIAL" device="UFIDUCIAL" value="FIDUCIALUFIDUCIAL"/>
 <part name="FD4" library="SparkFun-Aesthetics" deviceset="FIDUCIAL" device="UFIDUCIAL" value="FIDUCIALUFIDUCIAL"/>
-<part name="OUT" library="New_Parts_Connectors" deviceset="FPC_16_0.5MM" device="_BACKFLIP"/>
+<part name="OUT" library="SparkFun-Connectors" deviceset="CONN_16" device="FPC_16_0.5MM"/>
 <part name="SUPPLY22" library="SparkFun-PowerSymbols" deviceset="3.3V" device=""/>
 <part name="SUPPLY27" library="SparkFun-PowerSymbols" deviceset="V_USB" device=""/>
@@
 <part name="U$1" library="SparkX" deviceset="SPARKX-LOGO" device="3"/>
 <part name="LOGO3" library="SparkFun-Aesthetics" deviceset="OSHW-LOGO" device="MINI"/>
-<part name="IN" library="New_Parts_Connectors" deviceset="FPC_16_0.5MM" device="_BACKFLIP"/>
+<part name="IN" library="SparkFun-Connectors" deviceset="CONN_16" device="FPC_16_0.5MM"/>
 <part name="SUPPLY21" library="SparkFun-PowerSymbols" deviceset="3.3V" device=""/>
 <part name="SUPPLY25" library="SparkFun-PowerSymbols" deviceset="V_USB" device=""/>
@@
 <part name="C2" library="SparkFun-Capacitors" deviceset="0.1UF" device="-0402T-6.3V-10%-X7R" value="0.1uF"/>
 <part name="C4" library="SparkFun-Capacitors" deviceset="0.1UF" device="-0402T-6.3V-10%-X7R" value="0.1uF"/>
-<part name="R3" library="New-Parts_SparkFun-Resistors" deviceset="453KOHM" device="-0402T-1/16W-1%" value="453k"/>
-<part name="R1" library="New-Parts_SparkFun-Resistors" deviceset="1MOHM" device="-0402T-1/16W-1%" value="1M"/>
-<part name="R2" library="New-Parts_SparkFun-Resistors" deviceset="180KOHM" device="-0402T-1/16W-1%" value="180k"/>
+<part name="R3" library="SparkFun-Resistors" deviceset="453KOHM" device="-0402T-1/16W-1%" value="453k"/>
+<part name="R1" library="SparkFun-Resistors" deviceset="1MOHM" device="-0402T-1/16W-5%" value="1M"/>
+<part name="R2" library="SparkFun-Resistors" deviceset="180KOHM" device="-0402T-1/16W-1%" value="180k"/>
 <part name="GND2" library="SparkFun-PowerSymbols" deviceset="GND" device=""/>
 <part name="C1" library="SparkFun-Capacitors" deviceset="10UF" device="-0402T-6.3V-20%" value="10uF"/>
@@
 <instance part="FD4" gate="G$1" x="429.26" y="27.94" smashed="yes"/>
 <instance part="LOGO2" gate="G$1" x="307.34" y="25.4" smashed="yes"/>
-<instance part="OUT" gate="G$1" x="73.66" y="233.68" smashed="yes" rot="MR0">
-<attribute name="NAME" x="76.2" y="254.254" size="1.778" layer="95" rot="MR0"/>
-<attribute name="VALUE" x="76.2" y="208.28" size="1.778" layer="96" rot="MR0"/>
+<instance part="OUT" gate="G$1" x="76.2" y="231.14" smashed="yes" rot="R180">
+<attribute name="NAME" x="76.2" y="210.566" size="1.778" layer="95" rot="R180"/>
+<attribute name="VALUE" x="78.74" y="256.54" size="1.778" layer="96" rot="R180"/>
 </instance>
 <instance part="SUPPLY22" gate="G$1" x="63.5" y="254" smashed="yes">
@@
 <instance part="U$1" gate="G$1" x="307.34" y="7.62" smashed="yes"/>
 <instance part="LOGO3" gate="G$1" x="307.34" y="25.4" smashed="yes"/>
-<instance part="IN" gate="G$1" x="12.7" y="233.68" smashed="yes">
-<attribute name="NAME" x="10.16" y="254.254" size="1.778" layer="95"/>
-<attribute name="VALUE" x="10.16" y="208.28" size="1.778" layer="96"/>
+<instance part="IN" gate="G$1" x="10.16" y="231.14" smashed="yes" rot="MR180">
+<attribute name="NAME" x="10.16" y="210.566" size="1.778" layer="95" rot="MR180"/>
+<attribute name="VALUE" x="7.62" y="256.54" size="1.778" layer="96" rot="MR180"/>
 </instance>
 <instance part="SUPPLY21" gate="G$1" x="22.86" y="254" smashed="yes">
@@
 <segment>
 <pinref part="SUPPLY22" gate="G$1" pin="3.3V"/>
-<wire x1="63.5" y1="254" x2="63.5" y2="248.92" width="0.1524" layer="91"/>
 <pinref part="OUT" gate="G$1" pin="2"/>
-<wire x1="63.5" y1="248.92" x2="66.04" y2="248.92" width="0.1524" layer="91"/>
 <pinref part="OUT" gate="G$1" pin="15"/>
 <wire x1="66.04" y1="215.9" x2="63.5" y2="215.9" width="0.1524" layer="91"/>
 <wire x1="63.5" y1="215.9" x2="63.5" y2="248.92" width="0.1524" layer="91"/>
+<wire x1="63.5" y1="248.92" x2="63.5" y2="254" width="0.1524" layer="91"/>
+<wire x1="66.04" y1="248.92" x2="63.5" y2="248.92" width="0.1524" layer="91"/>
 <junction x="63.5" y="248.92"/>
 </segment>
 <segment>
 <pinref part="SUPPLY21" gate="G$1" pin="3.3V"/>
-<wire x1="22.86" y1="254" x2="22.86" y2="248.92" width="0.1524" layer="91"/>
 <pinref part="IN" gate="G$1" pin="2"/>
-<wire x1="22.86" y1="248.92" x2="20.32" y2="248.92" width="0.1524" layer="91"/>
 <pinref part="IN" gate="G$1" pin="15"/>
 <wire x1="20.32" y1="215.9" x2="22.86" y2="215.9" width="0.1524" layer="91"/>
 <wire x1="22.86" y1="215.9" x2="22.86" y2="248.92" width="0.1524" layer="91"/>
+<wire x1="22.86" y1="248.92" x2="22.86" y2="254" width="0.1524" layer="91"/>
+<wire x1="20.32" y1="248.92" x2="22.86" y2="248.92" width="0.1524" layer="91"/>
 <junction x="22.86" y="248.92"/>
 </segment>
@@
 <pinref part="IN" gate="G$1" pin="16"/>
 <wire x1="20.32" y1="213.36" x2="22.86" y2="213.36" width="0.1524" layer="91"/>
-<wire x1="22.86" y1="210.82" x2="22.86" y2="213.36" width="0.1524" layer="91"/>
-</segment>
-</net>
+<wire x1="22.86" y1="213.36" x2="22.86" y2="210.82" width="0.1524" layer="91"/>
+</segment>
+</net>
