File: Hardware/SparkX_smol_Power_AAA.brd (EAGLE design)
At the start: 10.7 x 40.6 mm, 47 parts, among them J3 AVR_SPI_PROG_3X2TESTPOINTS, U1 ATTINY43_QFN20, U2 TPS61200

Commit message: Update smôl logo
Parts:
- added U$13, U$14: SMOL_LOGOSMALL, SparkX:SMOL_SMALL
- moved U$3 0.19 mm to (5.33, 4.70)
Changed lines of the file:
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@@
 <wire x1="7.62" y1="31.75" x2="8.89" y2="31.75" width="0.3048" layer="21"/>
 <wire x1="8.255" y1="31.115" x2="8.255" y2="32.385" width="0.3048" layer="21"/>
-<polygon width="0.0762" layer="21">
-<vertex x="5.334" y="6.4135"/>
-<vertex x="2.794" y="5.3975"/>
-<vertex x="2.54" y="5.3975"/>
-<vertex x="4.572" y="7.1755"/>
-<vertex x="6.096" y="7.1755"/>
-<vertex x="8.128" y="5.3975"/>
-<vertex x="7.874" y="5.3975"/>
-</polygon>
-<polygon width="0.0762" layer="22">
-<vertex x="5.334" y="35.6235"/>
-<vertex x="2.794" y="34.6075"/>
-<vertex x="2.54" y="34.6075"/>
-<vertex x="4.572" y="36.3855"/>
-<vertex x="6.096" y="36.3855"/>
-<vertex x="8.128" y="34.6075"/>
-<vertex x="7.874" y="34.6075"/>
-</polygon>
 </plain>
 <attributes>
@@
 <element name="U$8" library="output" package="SM�L_POWER_AAA0" value="" x="1.0795" y="9.5885" smashed="yes" rot="R90"/>
 <element name="U$2" library="output" package="SM�L_POWER_AAA0" value="" x="5.334" y="25.4" smashed="yes" rot="MR0"/>
-<element name="U$3" library="output" package="OUT0" value="" x="5.334" y="4.8895" smashed="yes"/>
+<element name="U$3" library="output" package="OUT0" value="" x="5.334" y="4.699" smashed="yes"/>
 <element name="U$12" library="output" package="IN0" value="" x="5.334" y="34.3535" smashed="yes" rot="MR0"/>
+<element name="U$13" library="SparkX" package="SMOL_SMALL" value="SMOL_LOGOSMALL" x="5.334" y="6.604" smashed="yes"/>
+<element name="U$14" library="SparkX" package="SMOL_SMALL" value="SMOL_LOGOSMALL" x="5.334" y="35.814" smashed="yes" rot="MR0"/>
 </elements>
 <signals>
