File: Hardware/Production/SparkX_smol_Power_AAA-Panel.brd (EAGLE design)
At the start: 198.4 x 137.2 mm, 2166 parts, among them J10 AVR_SPI_PROG_3X2TESTPOINTS, J12 AVR_SPI_PROG_3X2TESTPOINTS, J14 AVR_SPI_PROG_3X2TESTPOINTS, J16 AVR_SPI_PROG_3X2TESTPOINTS, J18 AVR_SPI_PROG_3X2TESTPOINTS, J20 AVR_SPI_PROG_3X2TESTPOINTS, J22 AVR_SPI_PROG_3X2TESTPOINTS, J24 AVR_SPI_PROG_3X2TESTPOINTS, J26 AVR_SPI_PROG_3X2TESTPOINTS, J28 AVR_SPI_PROG_3X2TESTPOINTS, J3 AVR_SPI_PROG_3X2TESTPOINTS, J30 AVR_SPI_PROG_3X2TESTPOINTS, J32 AVR_SPI_PROG_3X2TESTPOINTS, J34 AVR_SPI_PROG_3X2TESTPOINTS, J36 AVR_SPI_PROG_3X2TESTPOINTS, J38 AVR_SPI_PROG_3X2TESTPOINTS, J4 AVR_SPI_PROG_3X2TESTPOINTS, J40 AVR_SPI_PROG_3X2TESTPOINTS, J42 AVR_SPI_PROG_3X2TESTPOINTS, J44 AVR_SPI_PROG_3X2TESTPOINTS, J46 AVR_SPI_PROG_3X2TESTPOINTS, J48 AVR_SPI_PROG_3X2TESTPOINTS, J50 AVR_SPI_PROG_3X2TESTPOINTS, J52 AVR_SPI_PROG_3X2TESTPOINTS, J54 AVR_SPI_PROG_3X2TESTPOINTS, J56 AVR_SPI_PROG_3X2TESTPOINTS, J58 AVR_SPI_PROG_3X2TESTPOINTS, J6 AVR_SPI_PROG_3X2TESTPOINTS, J60 AVR_SPI_PROG_3X2TESTPOINTS, J62 AVR_SPI_PROG_3X2TESTPOINTS, J64 AVR_SPI_PROG_3X2TESTPOINTS, J66 AVR_SPI_PROG_3X2TESTPOINTS, J68 AVR_SPI_PROG_3X2TESTPOINTS, J70 AVR_SPI_PROG_3X2TESTPOINTS, J72 AVR_SPI_PROG_3X2TESTPOINTS, J74 AVR_SPI_PROG_3X2TESTPOINTS, J76 AVR_SPI_PROG_3X2TESTPOINTS, J78 AVR_SPI_PROG_3X2TESTPOINTS, J8 AVR_SPI_PROG_3X2TESTPOINTS, J80 AVR_SPI_PROG_3X2TESTPOINTS, J82 AVR_SPI_PROG_3X2TESTPOINTS, J84 AVR_SPI_PROG_3X2TESTPOINTS, J86 AVR_SPI_PROG_3X2TESTPOINTS, J88 AVR_SPI_PROG_3X2TESTPOINTS, J90 AVR_SPI_PROG_3X2TESTPOINTS, J92 AVR_SPI_PROG_3X2TESTPOINTS, J94 AVR_SPI_PROG_3X2TESTPOINTS, J96 AVR_SPI_PROG_3X2TESTPOINTS, U1 ATTINY43_QFN20, U10 TPS61200, U11 ATTINY43_QFN20, U12 TPS61200, U13 ATTINY43_QFN20, U14 TPS61200, U15 ATTINY43_QFN20, U16 TPS61200, U17 ATTINY43_QFN20, U18 TPS61200, U19 ATTINY43_QFN20, U2 TPS61200, U20 TPS61200, U21 ATTINY43_QFN20, U22 TPS61200, U23 ATTINY43_QFN20, U24 TPS61200, U25 ATTINY43_QFN20, U26 TPS61200, U27 ATTINY43_QFN20, U28 TPS61200, U29 ATTINY43_QFN20, U3 ATTINY43_QFN20, U30 TPS61200, U31 ATTINY43_QFN20, U32 TPS61200, U33 ATTINY43_QFN20, U34 TPS61200, U35 ATTINY43_QFN20, U36 TPS61200, U37 ATTINY43_QFN20, U38 TPS61200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

Commit message: Update smôl logo
Parts:
- added U$625, U$626, U$640, U$641, U$655, U$656, U$670, U$671, U$685, U$686, U$700, U$701, U$715, U$716: (no value), output:SM�L_POWER_AAA0
- added U$627, U$642, U$657, U$672, U$687, U$702, U$717: (no value), output:OUT0
- added U$628, U$643, U$658, U$673, U$688, U$703, U$718: (no value), output:IN0
- added U$629, U$630, U$644, U$645, U$659, U$660, U$674, U$675, U$689, U$690, U$704, U$705, U$719, U$720: SMOL_LOGOSMALL, SparkX:SMOL_SMALL
- added U$631, U$632, U$646, U$647, U$661, U$662, U$676, U$677, U$691, U$692, U$706, U$707: SPARKX-LOGO3, SparkX:SPARKX-SMALL
- added U$633, U$648, U$663, U$678, U$693, U$708: (no value), output:#VIN#0
- added U$634, U$649, U$664, U$679, U$694, U$709: (no value), output:#3V3_EN#0
- added U$635, U$650, U$665, U$680, U$695, U$710: (no value), output:#PROC_PWR#0
- added U$636, U$651, U$666, U$681, U$696, U$711: (no value), output:#TXD#0
- added U$637, U$652, U$667, U$682, U$697, U$712: (no value), output:#RXD#0
- added U$638, U$653, U$668, U$683, U$698, U$713: (no value), output:5#5V0
- added U$639, U$654, U$669, U$684, U$699, U$714: (no value), output:MAX0
- U$100, U$191, U$295, U$386, U$490, U$581: device output:MAX0 -> output:SM�L_POWER_AAA0
- U$102, U$192, U$297, U$387, U$492, U$582: device output:SM�L_POWER_AAA0 -> output:OUT0
- U$103, U$298, U$493: device output:OUT0 -> output:IN0
- U$104, U$195, U$299, U$390, U$494, U$585: value (none) -> SMOL_LOGOSMALL; device output:IN0 -> SparkX:SMOL_SMALL
- U$105, U$119, U$13, U$14, U$209, U$210, U$300, U$314, U$404, U$405, U$495, U$509, U$599, U$600: value SPARKX-LOGO3 -> SMOL_LOGOSMALL; device SparkX:SPARKX-SMALL -> SparkX:SMOL_SMALL
- U$107, U$15, U$211, U$302, U$406, U$497, U$601: value (none) -> SPARKX-LOGO3; device output:#VIN#0 -> SparkX:SPARKX-SMALL
- U$108, U$303, U$498: device output:#3V3_EN#0 -> output:#VIN#0
- U$109, U$304, U$499: device output:#PROC_PWR#0 -> output:#3V3_EN#0
- U$110, U$305, U$500: device output:#TXD#0 -> output:#PROC_PWR#0
- U$111, U$306, U$501: device output:#RXD#0 -> output:#TXD#0
- U$112, U$307, U$502: device output:5#5V0 -> output:#RXD#0
- U$113, U$308, U$503: device output:MAX0 -> output:5#5V0
- U$114, U$219, U$24, U$309, U$414, U$504, U$609: device output:SM�L_POWER_AAA0 -> output:MAX0
- U$116, U$220, U$25, U$311, U$415, U$506, U$610: device output:OUT0 -> output:SM�L_POWER_AAA0
- U$117, U$312, U$507: device output:IN0 -> output:OUT0
- U$118, U$223, U$28, U$313, U$418, U$508, U$613: value SPARKX-LOGO3 -> (none); device SparkX:SPARKX-SMALL -> output:IN0
- U$120, U$224, U$29, U$315, U$419, U$510, U$614: value (none) -> SMOL_LOGOSMALL; device output:#VIN#0 -> SparkX:SMOL_SMALL
- U$121, U$16, U$212, U$316, U$407, U$511, U$602: value (none) -> SPARKX-LOGO3; device output:#3V3_EN#0 -> SparkX:SPARKX-SMALL
- U$122, U$226, U$31, U$317, U$421, U$512, U$616: value (none) -> SPARKX-LOGO3; device output:#PROC_PWR#0 -> SparkX:SPARKX-SMALL
- U$123, U$318, U$513: device output:#TXD#0 -> output:#VIN#0
- U$124, U$319, U$514: device output:#RXD#0 -> output:#3V3_EN#0
- U$125, U$320, U$515: device output:5#5V0 -> output:#PROC_PWR#0
- U$126, U$321, U$516: device output:MAX0 -> output:#TXD#0
- U$127, U$232, U$322, U$37, U$427, U$517, U$622: device output:SM�L_POWER_AAA0 -> output:#RXD#0
- U$128, U$218, U$23, U$323, U$413, U$518, U$608: device output:SM�L_POWER_AAA0 -> output:5#5V0
- U$129, U$324, U$519: device output:OUT0 -> output:MAX0
- U$130, U$221, U$26, U$325, U$416, U$520, U$611: device output:IN0 -> output:SM�L_POWER_AAA0
- U$131, U$145, U$235, U$236, U$326, U$340, U$40, U$41, U$430, U$431, U$521, U$535: value SPARKX-LOGO3 -> (none); device SparkX:SPARKX-SMALL -> output:SM�L_POWER_AAA0
- U$132, U$222, U$27, U$327, U$417, U$522, U$612: value SPARKX-LOGO3 -> (none); device SparkX:SPARKX-SMALL -> output:OUT0
- U$133, U$328, U$523: device output:#VIN#0 -> output:IN0
- U$134, U$225, U$30, U$329, U$420, U$524, U$615: value (none) -> SMOL_LOGOSMALL; device output:#3V3_EN#0 -> SparkX:SMOL_SMALL
- U$135, U$239, U$330, U$434, U$44, U$525: value (none) -> SMOL_LOGOSMALL; device output:#PROC_PWR#0 -> SparkX:SMOL_SMALL
- U$136, U$227, U$32, U$331, U$422, U$526, U$617: value (none) -> SPARKX-LOGO3; device output:#TXD#0 -> SparkX:SPARKX-SMALL
- U$137, U$241, U$332, U$436, U$46, U$527: value (none) -> SPARKX-LOGO3; device output:#RXD#0 -> SparkX:SPARKX-SMALL
- U$138, U$333, U$528: device output:5#5V0 -> output:#VIN#0
- U$139, U$334, U$529: device output:MAX0 -> output:#3V3_EN#0
- U$140, U$245, U$335, U$440, U$50, U$530: device output:SM�L_POWER_AAA0 -> output:#PROC_PWR#0
- U$141, U$231, U$336, U$36, U$426, U$531, U$621: device output:SM�L_POWER_AAA0 -> output:#TXD#0
- U$142, U$337, U$532: device output:OUT0 -> output:#RXD#0
- U$143, U$338, U$533: device output:IN0 -> output:5#5V0
- U$144, U$249, U$339, U$444, U$534, U$54: value SPARKX-LOGO3 -> (none); device SparkX:SPARKX-SMALL -> output:MAX0
- U$146, U$250, U$341, U$445, U$536, U$55: device output:#VIN#0 -> output:SM�L_POWER_AAA0
- U$147, U$342, U$537: device output:#3V3_EN#0 -> output:OUT0
- U$148, U$343, U$538: device output:#PROC_PWR#0 -> output:IN0
- U$149, U$240, U$344, U$435, U$45, U$539: value (none) -> SMOL_LOGOSMALL; device output:#TXD#0 -> SparkX:SMOL_SMALL
- U$150, U$254, U$345, U$449, U$540, U$59: value (none) -> SMOL_LOGOSMALL; device output:#RXD#0 -> SparkX:SMOL_SMALL
- U$151, U$242, U$346, U$437, U$47, U$541: value (none) -> SPARKX-LOGO3; device output:5#5V0 -> SparkX:SPARKX-SMALL
- U$152, U$256, U$347, U$451, U$542, U$61: value (none) -> SPARKX-LOGO3; device output:MAX0 -> SparkX:SPARKX-SMALL
- U$153, U$258, U$348, U$453, U$543, U$63: device output:SM�L_POWER_AAA0 -> output:#VIN#0
- U$154, U$244, U$349, U$439, U$49, U$544: device output:SM�L_POWER_AAA0 -> output:#3V3_EN#0
- U$155, U$350, U$545: device output:OUT0 -> output:#PROC_PWR#0
- U$156, U$351, U$546: device output:IN0 -> output:#TXD#0
- U$157, U$262, U$352, U$457, U$547, U$67: value SPARKX-LOGO3 -> (none); device SparkX:SPARKX-SMALL -> output:#RXD#0
- U$158, U$248, U$353, U$443, U$53, U$548: value SPARKX-LOGO3 -> (none); device SparkX:SPARKX-SMALL -> output:5#5V0
- U$159, U$354, U$549: device output:#VIN#0 -> output:MAX0
- U$160, U$251, U$355, U$446, U$550, U$56: device output:#3V3_EN#0 -> output:SM�L_POWER_AAA0
- U$161, U$265, U$356, U$460, U$551, U$70: device output:#PROC_PWR#0 -> output:SM�L_POWER_AAA0
- U$162, U$357, U$552: device output:#TXD#0 -> output:OUT0
- U$163, U$358, U$553: device output:#RXD#0 -> output:IN0
- U$164, U$255, U$359, U$450, U$554, U$60: value (none) -> SMOL_LOGOSMALL; device output:5#5V0 -> SparkX:SMOL_SMALL
- U$165, U$269, U$360, U$464, U$555, U$74: value (none) -> SMOL_LOGOSMALL; device output:MAX0 -> SparkX:SMOL_SMALL
- U$166, U$167, U$257, U$271, U$361, U$362, U$452, U$466, U$556, U$557, U$62, U$76: value (none) -> SPARKX-LOGO3; device output:SM�L_POWER_AAA0 -> SparkX:SPARKX-SMALL
- U$168, U$363, U$558: device output:OUT0 -> output:#VIN#0
- U$169, U$364, U$559: device output:IN0 -> output:#3V3_EN#0
- U$17, U$213, U$408, U$603: device output:#PROC_PWR#0 -> output:#VIN#0
- U$170, U$275, U$365, U$470, U$560, U$80: value SPARKX-LOGO3 -> (none); device SparkX:SPARKX-SMALL -> output:#PROC_PWR#0
- U$171, U$261, U$366, U$456, U$561, U$66: value SPARKX-LOGO3 -> (none); device SparkX:SPARKX-SMALL -> output:#TXD#0
- U$172, U$367, U$562: device output:#VIN#0 -> output:#RXD#0
- U$173, U$368, U$563: device output:#3V3_EN#0 -> output:5#5V0
- U$174, U$369, U$564: device output:#PROC_PWR#0 -> output:MAX0
- U$175, U$266, U$370, U$461, U$565, U$71: device output:#TXD#0 -> output:SM�L_POWER_AAA0
- U$176, U$280, U$371, U$475, U$566, U$85: device output:#RXD#0 -> output:SM�L_POWER_AAA0
- U$177, U$372, U$567: device output:5#5V0 -> output:OUT0
- U$178, U$373, U$568: device output:MAX0 -> output:IN0
- U$179, U$180, U$270, U$284, U$374, U$375, U$465, U$479, U$569, U$570, U$75, U$89: value (none) -> SMOL_LOGOSMALL; device output:SM�L_POWER_AAA0 -> SparkX:SMOL_SMALL
- U$18, U$214, U$409, U$604: device output:#TXD#0 -> output:#3V3_EN#0
- U$181, U$272, U$376, U$467, U$571, U$77: value (none) -> SPARKX-LOGO3; device output:OUT0 -> SparkX:SPARKX-SMALL
- U$182, U$286, U$377, U$481, U$572, U$91: value (none) -> SPARKX-LOGO3; device output:IN0 -> SparkX:SPARKX-SMALL
- U$183, U$288, U$378, U$483, U$573, U$93: value SPARKX-LOGO3 -> (none); device SparkX:SPARKX-SMALL -> output:#VIN#0
- U$184, U$274, U$379, U$469, U$574, U$79: value SPARKX-LOGO3 -> (none); device SparkX:SPARKX-SMALL -> output:#3V3_EN#0
- U$185, U$380, U$575: device output:#VIN#0 -> output:#PROC_PWR#0
- U$186, U$381, U$576: device output:#3V3_EN#0 -> output:#TXD#0
- U$187, U$382, U$577: device output:#PROC_PWR#0 -> output:#RXD#0
- U$188, U$383, U$578: device output:#TXD#0 -> output:5#5V0
- U$189, U$384, U$579: device output:#RXD#0 -> output:MAX0
- U$19, U$215, U$410, U$605: device output:#RXD#0 -> output:#PROC_PWR#0
- U$190, U$281, U$385, U$476, U$580, U$86: device output:5#5V0 -> output:SM�L_POWER_AAA0
- U$193, U$283, U$388, U$478, U$583, U$88: device output:SM�L_POWER_AAA0 -> output:IN0
- U$194, U$285, U$389, U$480, U$584, U$90: value (none) -> SMOL_LOGOSMALL; device output:OUT0 -> SparkX:SMOL_SMALL
- U$21, U$216, U$411, U$606: device output:5#5V0 -> output:#TXD#0
- U$217, U$22, U$412, U$607: device output:MAX0 -> output:#RXD#0
- U$228, U$33, U$423, U$618: device output:#RXD#0 -> output:#VIN#0
- U$229, U$34, U$424, U$619: device output:5#5V0 -> output:#3V3_EN#0
- U$230, U$35, U$425, U$620: device output:MAX0 -> output:#PROC_PWR#0
- U$233, U$38, U$428, U$623: device output:OUT0 -> output:5#5V0
- U$234, U$39, U$429, U$624: device output:IN0 -> output:MAX0
- U$237, U$42, U$432: device output:#VIN#0 -> output:OUT0
- U$238, U$43, U$433: device output:#3V3_EN#0 -> output:IN0
- U$243, U$438, U$48: device output:MAX0 -> output:#VIN#0
- U$246, U$441, U$51: device output:OUT0 -> output:#TXD#0
- U$247, U$442, U$52: device output:IN0 -> output:#RXD#0
- U$252, U$447, U$57: device output:#PROC_PWR#0 -> output:OUT0
- U$253, U$448, U$58: device output:#TXD#0 -> output:IN0
- U$259, U$454, U$64: device output:OUT0 -> output:#3V3_EN#0
- U$260, U$455, U$65: device output:IN0 -> output:#PROC_PWR#0
- U$263, U$458, U$68: device output:#VIN#0 -> output:5#5V0
- U$264, U$459, U$69: device output:#3V3_EN#0 -> output:MAX0
- U$267, U$462, U$72: device output:#RXD#0 -> output:OUT0
- U$268, U$463, U$73: device output:5#5V0 -> output:IN0
- U$273, U$468, U$78: device output:IN0 -> output:#VIN#0
- U$276, U$471, U$81: device output:#VIN#0 -> output:#TXD#0
- U$277, U$472, U$82: device output:#3V3_EN#0 -> output:#RXD#0
- U$278, U$473, U$83: device output:#PROC_PWR#0 -> output:5#5V0
- U$279, U$474, U$84: device output:#TXD#0 -> output:MAX0
- U$282, U$477, U$87: device output:MAX0 -> output:OUT0
- U$289, U$484, U$94: device output:#VIN#0 -> output:#3V3_EN#0
- U$290, U$485, U$95: device output:#3V3_EN#0 -> output:#PROC_PWR#0
- U$291, U$486, U$96: device output:#PROC_PWR#0 -> output:#TXD#0
- U$292, U$487, U$97: device output:#TXD#0 -> output:#RXD#0
- U$293, U$488, U$98: device output:#RXD#0 -> output:5#5V0
- U$294, U$489, U$99: device output:5#5V0 -> output:MAX0
- moved U$215 170.9 mm to (160.9, 3.75)
- moved U$214 170.5 mm to (163.5, 14.0)
- moved U$228 168.0 mm to (170.5, 7.62)
- moved U$234 166.6 mm to (176.6, 29.5), flipped to the top
- moved U$230 166.0 mm to (172.1, 3.75), flipped to the bottom
- moved U$218 165.6 mm to (165.4, 30.4), turned to 0 degrees
- moved U$229 164.9 mm to (174.7, 14.0), flipped to the bottom
- moved U$227 164.6 mm to (173.0, 27.6)
- moved U$219 164.3 mm to (165.4, 29.5), flipped to the top
- moved U$221 164.3 mm to (161.8, 25.4)
- moved U$233 160.8 mm to (176.6, 30.4)
- moved U$231 160.3 mm to (171.6, 33.0), flipped to the bottom, turned to 0 degrees
- moved U$213 159.3 mm to (159.3, 7.62)
- moved U$232 159.3 mm to (171.6, 30.5)
- moved U$222 159.2 mm to (161.8, 4.70), turned to 0 degrees
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